Commit message: Update frame imu

File: limo_description/urdf/limo_ackerman.xacro (robot description, xacro)
@@ -60,5 +60,5 @@
     </xacro:limo_depth_camera>
     <xacro:limo_imu parent_prefix="base_link" frame_prefix="imu">
-        <origin xyz="0.0 0 -0.1" rpy="0 0 0"/>
+        <origin xyz="${-wheelbase/2} 0 ${wheel_vertical_offset}" rpy="0 0 0"/>
     </xacro:limo_imu>
     <xacro:limo_left_steering_hinge parent_prefix="base_link" wheel_prefix="left_steering_hinge">

Commit message: Add stanley control

File: limo_description/urdf/limo_ackerman.xacro (robot description, xacro)
@@ -6,14 +6,4 @@
     <!-- <xacro:include filename="$(find limo_description)/urdf/limo_ackerman.gazebo" /> -->
     <xacro:include filename="$(find limo_description)/urdf/gazebo_control.xacro" />
-    <!-- inertial_cylinder -->
-    <xacro:macro name="inertial_cylinder" params="mass length radius *origin">
-        <inertial>
-            <xacro:insert_block name="origin"/>
-            <mass value="${mass}" />
-            <inertia ixx="${(1/12) * mass * (3*radius*radius + length*length)}" ixy="0.0" ixz="0.0"
-                    iyy="${(1/12) * mass * (3*radius*radius + length*length)}" iyz="0.0"
-                    izz="${(1/2) * mass * (radius*radius)}" />
-        </inertial>
-    </xacro:macro>
     <!-- Variables -->
     <xacro:property name="M_PI" value="3.14159"/>
