Commit message: add steering pose and wheel velo controller

File: limo_description/urdf/gazebo_control.xacro (robot description, xacro)
@@ -36,4 +36,30 @@
               <state_interface name="effort"/>
         </joint>
+        <joint name="left_steering_hinge_wheel">
+            <command_interface name="position">
+                <param name="min">-0.523598767</param>
+                <param name="max">0.523598767</param>
+              </command_interface>
+              <state_interface name="position">
+                <param name="initial_value">0.0</param>
+              </state_interface>
+              <state_interface name="velocity">
+                <param name="initial_value">0.0</param>
+              </state_interface>
+              <state_interface name="effort"/>
+        </joint>
+        <joint name="right_steering_hinge_wheel">
+            <command_interface name="position">
+                <param name="min">-0.523598767</param>
+                <param name="max">0.523598767</param>
+              </command_interface>
+              <state_interface name="position">
+                <param name="initial_value">0.0</param>
+              </state_interface>
+              <state_interface name="velocity">
+                <param name="initial_value">0.0</param>
+              </state_interface>
+              <state_interface name="effort"/>
+        </joint>
     </ros2_control>
     <gazebo reference="base_link">
@@ -41,7 +67,6 @@
         <kp  value="10000000.0"/>
         <kd  value="1.0"/>
-        <material>Gazebo/Green</material>
     </gazebo>
-    <gazebo reference="front_left_wheel">
+    <gazebo reference="front_left_wheel_link">
         <mu1>10.0</mu1>
         <mu2>10.0</mu2>
@@ -50,5 +75,5 @@
         <kd  value="1.0"/>
     </gazebo>
-    <gazebo reference="front_right_wheel">
+    <gazebo reference="front_right_wheel_link">
         <mu1>10.0</mu1>
         <mu2>10.0</mu2>

Commit message: Add 3 model odom and ground truth

File: limo_description/urdf/gazebo_control.xacro (robot description, xacro)
@@ -9,4 +9,17 @@
         <plugin filename="libgazebo_ros2_control.so" name="gazebo_ros2_control">
             <parameters>$(find limo_description)/config/gazebo_controllers.yaml</parameters>
+        </plugin>
+        <plugin name="gazebo_ros_p3d" filename="libgazebo_ros_p3d.so">
+            <ros>
+                <!-- The topic name where the position will be published -->
+                <remapping>odom:=/odometry/gt</remapping>
+            </ros>
+            <frame_name>odom</frame_name>
+            <!-- Replace with your robot's main link -->
+            <body_name>base_footprint</body_name>
+            <!-- Update rate in Hz -->
+            <update_rate>100.0</update_rate>
+            <xyz_offset>-9.5 0.0 0.0</xyz_offset>
+            <rpy_offset>0.0 0.0 1.5708</rpy_offset>
         </plugin>
     </gazebo>

File: limo_description/urdf/limo_ackerman.xacro (robot description, xacro)
@@ -60,5 +60,5 @@
     </xacro:limo_depth_camera>
     <xacro:limo_imu parent_prefix="base_link" frame_prefix="imu">
-        <origin xyz="${-wheelbase/2} 0 ${wheel_vertical_offset}" rpy="0 0 0"/>
+        <origin xyz="0.0 0 -0.1" rpy="0 0 0"/>
     </xacro:limo_imu>
     <xacro:limo_left_steering_hinge parent_prefix="base_link" wheel_prefix="left_steering_hinge">

Commit message: fix Single-Track

File: limo_description/urdf/gazebo_control.xacro (robot description, xacro)
@@ -80,4 +80,17 @@
               <state_interface name="effort"/>
         </joint>
+        <joint name="steering">
+            <command_interface name="position">
+                <param name="min">-0.523598767</param>
+                <param name="max">0.523598767</param>
+              </command_interface>
+              <state_interface name="position">
+                <param name="initial_value">0.0</param>
+              </state_interface>
+              <state_interface name="velocity">
+                <param name="initial_value">0.0</param>
+              </state_interface>
+              <state_interface name="effort"/>
+        </joint>
     </ros2_control>
     <gazebo reference="base_link">

File: limo_description/urdf/limo_ackerman.xacro (robot description, xacro)
@@ -6,4 +6,14 @@
     <!-- <xacro:include filename="$(find limo_description)/urdf/limo_ackerman.gazebo" /> -->
     <xacro:include filename="$(find limo_description)/urdf/gazebo_control.xacro" />
+    <!-- inertial_cylinder -->
+    <xacro:macro name="inertial_cylinder" params="mass length radius *origin">
+        <inertial>
+            <xacro:insert_block name="origin"/>
+            <mass value="${mass}" />
+            <inertia ixx="${(1/12) * mass * (3*radius*radius + length*length)}" ixy="0.0" ixz="0.0"
+                    iyy="${(1/12) * mass * (3*radius*radius + length*length)}" iyz="0.0"
+                    izz="${(1/2) * mass * (radius*radius)}" />
+        </inertial>
+    </xacro:macro>
     <!-- Variables -->
     <xacro:property name="M_PI" value="3.14159"/>
@@ -118,3 +128,30 @@
         <axis xyz="0 -1 0"/>
     </joint>
+    <!-- Steer Link -->
+    <link name="steer_link">
+        <visual>
+            <origin xyz="0 0 0" rpy="0 0 0"/>
+            <geometry>
+                <cylinder length="0.002" radius="0.001"/>
+            </geometry>
+        </visual>
+        <collision>
+            <origin xyz="0 0 0" rpy="0 0 0" />
+          <geometry>
+              <cylinder length="0.002" radius="0.001"/>
+          </geometry>
+        </collision>
+        <xacro:inertial_cylinder mass="0.001" length="0.002" radius="0.001">
+            <origin xyz="0 0 0" rpy="0 0 0"/>
+        </xacro:inertial_cylinder>
+    </link>
+    <joint name="steering" type="revolute">
+        <parent link="base_link"/>
+        <child link="steer_link"/>
+        <origin xyz="${wheelbase/2} 0 ${wheel_vertical_offset}" rpy="0 0 0" />
+        <axis xyz="0 0 1" />
+        <limit lower="-0.523598767" upper="0.523598767" effort="5" velocity="0.5" />
+        <dynamics damping="1.0" friction="2.0"/>
+    </joint>
+    <!-- Steer Link -->
 </robot>

Commit message: Add delta_steering in odom_cal and add param to change mode in controller_server

File: limo_description/urdf/gazebo_control.xacro (robot description, xacro)
@@ -81,17 +81,4 @@
               <state_interface name="effort"/>
         </joint>
-        <joint name="steering">
-            <command_interface name="position">
-                <param name="min">-0.523598767</param>
-                <param name="max">0.523598767</param>
-              </command_interface>
-              <state_interface name="position">
-                <param name="initial_value">0.0</param>
-              </state_interface>
-              <state_interface name="velocity">
-                <param name="initial_value">0.0</param>
-              </state_interface>
-              <state_interface name="effort"/>
-        </joint>
     </ros2_control>
     <gazebo reference="base_link">

File: limo_description/urdf/limo_ackerman.xacro (robot description, xacro)
@@ -128,30 +128,3 @@
         <axis xyz="0 -1 0"/>
     </joint>
-    <!-- Steer Link -->
-    <link name="steer_link">
-        <visual>
-            <origin xyz="0 0 0" rpy="0 0 0"/>
-            <geometry>
-                <cylinder length="0.002" radius="0.001"/>
-            </geometry>
-        </visual>
-        <collision>
-            <origin xyz="0 0 0" rpy="0 0 0" />
-          <geometry>
-              <cylinder length="0.002" radius="0.001"/>
-          </geometry>
-        </collision>
-        <xacro:inertial_cylinder mass="0.001" length="0.002" radius="0.001">
-            <origin xyz="0 0 0" rpy="0 0 0"/>
-        </xacro:inertial_cylinder>
-    </link>
-    <joint name="steering" type="revolute">
-        <parent link="base_link"/>
-        <child link="steer_link"/>
-        <origin xyz="${wheelbase/2} 0 ${wheel_vertical_offset}" rpy="0 0 0" />
-        <axis xyz="0 0 1" />
-        <limit lower="-0.523598767" upper="0.523598767" effort="5" velocity="0.5" />
-        <dynamics damping="1.0" friction="2.0"/>
-    </joint>
-    <!-- Steer Link -->
 </robot>

Commit message: EKF update

File: limo_description/urdf/gazebo_control.xacro (robot description, xacro)
@@ -81,4 +81,17 @@
               <state_interface name="effort"/>
         </joint>
+        <joint name="steering">
+            <command_interface name="position">
+                <param name="min">-0.523598767</param>
+                <param name="max">0.523598767</param>
+              </command_interface>
+              <state_interface name="position">
+                <param name="initial_value">0.0</param>
+              </state_interface>
+              <state_interface name="velocity">
+                <param name="initial_value">0.0</param>
+              </state_interface>
+              <state_interface name="effort"/>
+        </joint>
     </ros2_control>
     <gazebo reference="base_link">

File: limo_description/urdf/limo_ackerman.xacro (robot description, xacro)
@@ -128,3 +128,30 @@
         <axis xyz="0 -1 0"/>
     </joint>
+    <!-- Steer Link -->
+    <link name="steer_link">
+        <visual>
+            <origin xyz="0 0 0" rpy="0 0 0"/>
+            <geometry>
+                <cylinder length="0.002" radius="0.001"/>
+            </geometry>
+        </visual>
+        <collision>
+            <origin xyz="0 0 0" rpy="0 0 0" />
+          <geometry>
+              <cylinder length="0.002" radius="0.001"/>
+          </geometry>
+        </collision>
+        <xacro:inertial_cylinder mass="0.001" length="0.002" radius="0.001">
+            <origin xyz="0 0 0" rpy="0 0 0"/>
+        </xacro:inertial_cylinder>
+    </link>
+    <joint name="steering" type="revolute">
+        <parent link="base_link"/>
+        <child link="steer_link"/>
+        <origin xyz="${wheelbase/2} 0 ${wheel_vertical_offset}" rpy="0 0 0" />
+        <axis xyz="0 0 1" />
+        <limit lower="-0.523598767" upper="0.523598767" effort="5" velocity="0.5" />
+        <dynamics damping="1.0" friction="2.0"/>
+    </joint>
+    <!-- Steer Link -->
 </robot>

Commit message: add slip in basic.world and fix base footprint

File: limo_description/urdf/gazebo_control.xacro (robot description, xacro)
@@ -81,21 +81,21 @@
     </ros2_control>
     <gazebo reference="base_link">
-        <minDepth>0.001</minDepth>
-        <kp  value="10000000.0"/>
-        <kd  value="1.0"/>
+      <minDepth>0.001</minDepth>
+      <kp  value="10000000.0"/>
+      <kd  value="1.0"/>
     </gazebo>
     <gazebo reference="front_left_wheel_link">
-        <mu1>10.0</mu1>
-        <mu2>10.0</mu2>
-        <minDepth>0.001</minDepth>
-        <kp  value="10000000.0"/>
-        <kd  value="1.0"/>
+      <mu1>10.0</mu1>
+      <mu2>10.0</mu2>
+      <minDepth>0.001</minDepth>
+      <kp  value="10000000.0"/>
+      <kd  value="1.0"/>
     </gazebo>
     <gazebo reference="front_right_wheel_link">
-        <mu1>10.0</mu1>
-        <mu2>10.0</mu2>
-        <minDepth>0.001</minDepth>
-        <kp  value="1000000.0"/>
-        <kd  value="1.0"/>
+      <mu1>10.0</mu1>
+      <mu2>10.0</mu2>
+      <minDepth>0.001</minDepth>
+      <kp  value="1000000.0"/>
+      <kd  value="1.0"/>
     </gazebo>
 </robot>

File: limo_description/urdf/limo_ackerman.xacro (robot description, xacro)
@@ -20,12 +20,12 @@
     <link name="base_footprint"/>
     <joint name="base_joint" type="fixed">
-    <parent link="base_footprint"/>
-    <child link="base_link"/>
-    <origin xyz="0.0 0.0 0.15" rpy="0 0 0"/>
+        <parent link="base_footprint"/>
+        <child link="base_link"/>
+        <origin xyz="0.0 0.0 0.15" rpy="0 0 0"/>
     </joint>
     <!-- Base link -->
     <link name="base_link">
         <visual>
-            <origin xyz="0 0 -0.15" rpy="0 0 1.57" />
+            <origin xyz="${wheelbase/2} 0 -0.15" rpy="0 0 1.57" />
             <geometry>
                 <mesh filename="file:///$(find limo_description)/meshes/limo_base.dae" />
@@ -33,5 +33,5 @@
         </visual>
         <collision>
-            <origin xyz="0 0 0" rpy="0 0 0" />
+            <origin xyz="${wheelbase/2} 0 0" rpy="0 0 0" />
           <geometry>
               <box size="${base_x_size} ${base_y_size} ${base_z_size}"/>
@@ -54,8 +54,8 @@
     </joint>
     <xacro:limo_laser parent_prefix="base_link" frame_prefix="laser">
-        <origin xyz="0.103 0 -0.034" rpy="0 0 0"/>
+        <origin xyz="${wheelbase/2 + 0.103} 0 -0.034" rpy="0 0 0"/>
     </xacro:limo_laser>
     <xacro:limo_depth_camera parent_prefix="base_link" frame_prefix="depth_camera">
-        <origin xyz="0.084 0 0.03" rpy="0 0 0"/>
+        <origin xyz="${wheelbase/2 + 0.084} 0 0.03" rpy="0 0 0"/>
     </xacro:limo_depth_camera>
     <xacro:limo_imu parent_prefix="base_link" frame_prefix="imu">
@@ -63,8 +63,8 @@
     </xacro:limo_imu>
     <xacro:limo_left_steering_hinge parent_prefix="base_link" wheel_prefix="left_steering_hinge">
-        <origin xyz="${wheelbase/2} ${track/2} ${wheel_vertical_offset}" rpy="0 0  0" />
+        <origin xyz="${wheelbase} ${track/2} ${wheel_vertical_offset}" rpy="0 0  0" />
     </xacro:limo_left_steering_hinge>
     <xacro:limo_right_steering_hinge parent_prefix="base_link" wheel_prefix="right_steering_hinge">
-        <origin xyz="${wheelbase/2} ${-track/2} ${wheel_vertical_offset}" rpy="${M_PI} 0 0" />
+        <origin xyz="${wheelbase} ${-track/2} ${wheel_vertical_offset}" rpy="${M_PI} 0 0" />
     </xacro:limo_right_steering_hinge>
     <link name="rear_left_wheel_link">
@@ -90,5 +90,5 @@
         <parent link="base_link"/>
         <child link="rear_left_wheel_link"/>
-        <origin xyz="${-wheelbase/2} ${track/2} ${wheel_vertical_offset}" rpy="0 0 0" />
+        <origin xyz="0 ${track/2} ${wheel_vertical_offset}" rpy="0 0 0" />
         <axis xyz="0 1 0"/>
     </joint>
@@ -115,5 +115,5 @@
         <parent link="base_link"/>
         <child link="rear_right_wheel_link"/>
-        <origin xyz="${-wheelbase/2} ${-track/2} ${wheel_vertical_offset}" rpy="${M_PI} 0 0" />
+        <origin xyz="0 ${-track/2} ${wheel_vertical_offset}" rpy="${M_PI} 0 0" />
         <axis xyz="0 -1 0"/>
     </joint>

Commit message: update plotter and mu in urdf

File: limo_description/urdf/gazebo_control.xacro (robot description, xacro)
@@ -81,21 +81,21 @@
     </ros2_control>
     <gazebo reference="base_link">
-      <minDepth>0.001</minDepth>
-      <kp  value="10000000.0"/>
-      <kd  value="1.0"/>
+        <minDepth>0.001</minDepth>
+        <kp  value="10000000.0"/>
+        <kd  value="1.0"/>
     </gazebo>
     <gazebo reference="front_left_wheel_link">
-      <mu1>10.0</mu1>
-      <mu2>10.0</mu2>
-      <minDepth>0.001</minDepth>
-      <kp  value="10000000.0"/>
-      <kd  value="1.0"/>
+        <mu1>10.0</mu1>
+        <mu2>10.0</mu2>
+        <minDepth>0.001</minDepth>
+        <kp  value="10000000.0"/>
+        <kd  value="1.0"/>
     </gazebo>
     <gazebo reference="front_right_wheel_link">
-      <mu1>10.0</mu1>
-      <mu2>10.0</mu2>
-      <minDepth>0.001</minDepth>
-      <kp  value="1000000.0"/>
-      <kd  value="1.0"/>
+        <mu1>10.0</mu1>
+        <mu2>10.0</mu2>
+        <minDepth>0.001</minDepth>
+        <kp  value="1000000.0"/>
+        <kd  value="1.0"/>
     </gazebo>
 </robot>

File: limo_description/urdf/limo_ackerman.xacro (robot description, xacro)
@@ -20,12 +20,12 @@
     <link name="base_footprint"/>
     <joint name="base_joint" type="fixed">
-        <parent link="base_footprint"/>
-        <child link="base_link"/>
-        <origin xyz="0.0 0.0 0.15" rpy="0 0 0"/>
+    <parent link="base_footprint"/>
+    <child link="base_link"/>
+    <origin xyz="0.0 0.0 0.15" rpy="0 0 0"/>
     </joint>
     <!-- Base link -->
     <link name="base_link">
         <visual>
-            <origin xyz="${wheelbase/2} 0 -0.15" rpy="0 0 1.57" />
+            <origin xyz="0 0 -0.15" rpy="0 0 1.57" />
             <geometry>
                 <mesh filename="file:///$(find limo_description)/meshes/limo_base.dae" />
@@ -33,5 +33,5 @@
         </visual>
         <collision>
-            <origin xyz="${wheelbase/2} 0 0" rpy="0 0 0" />
+            <origin xyz="0 0 0" rpy="0 0 0" />
           <geometry>
               <box size="${base_x_size} ${base_y_size} ${base_z_size}"/>
@@ -54,8 +54,8 @@
     </joint>
     <xacro:limo_laser parent_prefix="base_link" frame_prefix="laser">
-        <origin xyz="${wheelbase/2 + 0.103} 0 -0.034" rpy="0 0 0"/>
+        <origin xyz="0.103 0 -0.034" rpy="0 0 0"/>
     </xacro:limo_laser>
     <xacro:limo_depth_camera parent_prefix="base_link" frame_prefix="depth_camera">
-        <origin xyz="${wheelbase/2 + 0.084} 0 0.03" rpy="0 0 0"/>
+        <origin xyz="0.084 0 0.03" rpy="0 0 0"/>
     </xacro:limo_depth_camera>
     <xacro:limo_imu parent_prefix="base_link" frame_prefix="imu">
@@ -63,8 +63,8 @@
     </xacro:limo_imu>
     <xacro:limo_left_steering_hinge parent_prefix="base_link" wheel_prefix="left_steering_hinge">
-        <origin xyz="${wheelbase} ${track/2} ${wheel_vertical_offset}" rpy="0 0  0" />
+        <origin xyz="${wheelbase/2} ${track/2} ${wheel_vertical_offset}" rpy="0 0  0" />
     </xacro:limo_left_steering_hinge>
     <xacro:limo_right_steering_hinge parent_prefix="base_link" wheel_prefix="right_steering_hinge">
-        <origin xyz="${wheelbase} ${-track/2} ${wheel_vertical_offset}" rpy="${M_PI} 0 0" />
+        <origin xyz="${wheelbase/2} ${-track/2} ${wheel_vertical_offset}" rpy="${M_PI} 0 0" />
     </xacro:limo_right_steering_hinge>
     <link name="rear_left_wheel_link">
@@ -85,4 +85,12 @@
               <cylinder length="${wheel_length}" radius="${wheel_radius}" />
           </geometry>
+          <surface>
+            <friction>
+                <ode>
+                    <mu>10.0</mu>
+                    <mu2>10.0</mu2>
+                </ode>
+            </friction>
+          </surface>
         </collision>
     </link>
@@ -90,5 +98,5 @@
         <parent link="base_link"/>
         <child link="rear_left_wheel_link"/>
-        <origin xyz="0 ${track/2} ${wheel_vertical_offset}" rpy="0 0 0" />
+        <origin xyz="${-wheelbase/2} ${track/2} ${wheel_vertical_offset}" rpy="0 0 0" />
         <axis xyz="0 1 0"/>
     </joint>
@@ -110,4 +118,12 @@
                   <cylinder length="${wheel_length}" radius="${wheel_radius}" />
               </geometry>
+              <surface>
+               <friction>
+                   <ode>
+                     <mu>10.0</mu>
+                     <mu2>10.0</mu2>
+                   </ode>
+               </friction>
+              </surface>
             </collision>
         </link>
@@ -115,5 +131,5 @@
         <parent link="base_link"/>
         <child link="rear_right_wheel_link"/>
-        <origin xyz="0 ${-track/2} ${wheel_vertical_offset}" rpy="${M_PI} 0 0" />
+        <origin xyz="${-wheelbase/2} ${-track/2} ${wheel_vertical_offset}" rpy="${M_PI} 0 0" />
         <axis xyz="0 -1 0"/>
     </joint>

File: limo_description/urdf/limo_steering_hinge.xacro (robot description, xacro)
@@ -46,4 +46,12 @@
                 <cylinder length="${wheel_length}" radius="${wheel_radius}" />
             </geometry>
+            <surface>
+              <friction>
+                <ode>
+                  <mu>10.0</mu>
+                  <mu2>10.0</mu2>
+                </ode>
+              </friction>
+            </surface>
           </collision>
       </link>
@@ -100,4 +108,12 @@
                 <cylinder length="${wheel_length}" radius="${wheel_radius}" />
             </geometry>
+            <surface>
+              <friction>
+                <ode>
+                  <mu>10.0</mu>
+                  <mu2>10.0</mu2>
+                </ode>
+              </friction>
+            </surface>
           </collision>
       </link>
