Commit message: Update new urdf

File: limo_description/urdf/gazebo_control.xacro (robot description, xacro)
@@ -29,27 +29,27 @@
         <joint name="rear_left_wheel">
             <command_interface name="velocity">
-                <param name="min">-5</param>
-                <param name="max">5</param>
-              </command_interface>
-              <state_interface name="position">
-                <param name="initial_value">0.0</param>
-              </state_interface>
-              <state_interface name="velocity">
-                <param name="initial_value">0.0</param>
-              </state_interface>
-              <state_interface name="effort"/>
+                <param name="min">-20</param>
+                <param name="max">20</param>
+            </command_interface>
+            <state_interface name="position">
+              <param name="initial_value">0.0</param>
+            </state_interface>
+            <state_interface name="velocity">
+              <param name="initial_value">0.0</param>
+            </state_interface>
+            <state_interface name="effort"/>
         </joint>
         <joint name="rear_right_wheel">
             <command_interface name="velocity">
-                <param name="min">-5</param>
-                <param name="max">5</param>
-              </command_interface>
-              <state_interface name="position">
-                <param name="initial_value">0.0</param>
-              </state_interface>
-              <state_interface name="velocity">
-                <param name="initial_value">0.0</param>
-              </state_interface>
-              <state_interface name="effort"/>
+                <param name="min">-20</param>
+                <param name="max">20</param>
+            </command_interface>
+            <state_interface name="position">
+              <param name="initial_value">0.0</param>
+            </state_interface>
+            <state_interface name="velocity">
+              <param name="initial_value">0.0</param>
+            </state_interface>
+            <state_interface name="effort"/>
         </joint>
         <joint name="left_steering_hinge_wheel">
@@ -57,12 +57,12 @@
                 <param name="min">-0.523598767</param>
                 <param name="max">0.523598767</param>
-              </command_interface>
-              <state_interface name="position">
-                <param name="initial_value">0.0</param>
-              </state_interface>
-              <state_interface name="velocity">
-                <param name="initial_value">0.0</param>
-              </state_interface>
-              <state_interface name="effort"/>
+            </command_interface>
+            <state_interface name="position">
+              <param name="initial_value">0.0</param>
+            </state_interface>
+            <state_interface name="velocity">
+              <param name="initial_value">0.0</param>
+            </state_interface>
+            <state_interface name="effort"/>
         </joint>
         <joint name="right_steering_hinge_wheel">
@@ -70,32 +70,75 @@
                 <param name="min">-0.523598767</param>
                 <param name="max">0.523598767</param>
-              </command_interface>
-              <state_interface name="position">
+            </command_interface>
+            <state_interface name="position">
+              <param name="initial_value">0.0</param>
+            </state_interface>
+            <state_interface name="velocity">
+              <param name="initial_value">0.0</param>
+            </state_interface>
+            <state_interface name="effort"/>
+        </joint>
+        <joint name="front_left_wheel">
+            <command_interface name="velocity"/>
+            <state_interface name="position">
                 <param name="initial_value">0.0</param>
-              </state_interface>
-              <state_interface name="velocity">
+            </state_interface>
+            <state_interface name="velocity"/>
+            <state_interface name="effort"/>
+        </joint>
+        <joint name="front_right_wheel">
+            <command_interface name="velocity"/>
+            <state_interface name="position">
                 <param name="initial_value">0.0</param>
-              </state_interface>
-              <state_interface name="effort"/>
+            </state_interface>
+            <state_interface name="velocity"/>
+            <state_interface name="effort"/>
         </joint>
     </ros2_control>
+    <gazebo>
+        <mu1 value="10"/>
+        <mu2 value="10"/>
+        <kp value="10000000.0" />
+        <kd value="0" />
+        <fdir1 value="1 0 0"/>
+        <minDepth value="0.001" />
+        <maxContacts value="64"/>
+    </gazebo>
     <gazebo reference="base_link">
         <minDepth>0.001</minDepth>
         <kp  value="10000000.0"/>
-        <kd  value="1.0"/>
+        <kd  value="0"/>
     </gazebo>
     <gazebo reference="front_left_wheel_link">
+        <material>Gazebo/Black</material>
         <mu1>10.0</mu1>
         <mu2>10.0</mu2>
         <minDepth>0.001</minDepth>
         <kp  value="10000000.0"/>
-        <kd  value="1.0"/>
+        <kd  value="0"/>
     </gazebo>
     <gazebo reference="front_right_wheel_link">
+        <material>Gazebo/Black</material>
         <mu1>10.0</mu1>
         <mu2>10.0</mu2>
         <minDepth>0.001</minDepth>
-        <kp  value="1000000.0"/>
-        <kd  value="1.0"/>
+        <kp  value="10000000.0"/>
+        <kd  value="0"/>
+    </gazebo>
+    <gazebo reference="rear_left_wheel_link">
+        <material>Gazebo/Black</material>
+        <mu1>10.0</mu1>
+        <mu2>10.0</mu2>
+        <minDepth>0.001</minDepth>
+        <kp  value="10000000.0"/>
+        <kd  value="0"/>
+    </gazebo>
+    <gazebo reference="rear_right_wheel_link">
+        <material>Gazebo/Black</material>
+        <mu1>10.0</mu1>
+        <mu2>10.0</mu2>
+        <minDepth>0.001</minDepth>
+        <kp  value="10000000.0"/>
+        <kd  value="0"/>
     </gazebo>
 </robot>

Commit message: Fix odom

File: limo_description/urdf/gazebo_control.xacro (robot description, xacro)
@@ -100,5 +100,5 @@
         <mu2 value="10"/>
         <kp value="10000000.0" />
-        <kd value="0" />
+        <kd value="0"/>
         <fdir1 value="1 0 0"/>
         <minDepth value="0.001" />
@@ -108,5 +108,5 @@
         <minDepth>0.001</minDepth>
         <kp  value="10000000.0"/>
-        <kd  value="0"/>
+        <kd value="0"/>
     </gazebo>
     <gazebo reference="front_left_wheel_link">
@@ -116,5 +116,5 @@
         <minDepth>0.001</minDepth>
         <kp  value="10000000.0"/>
-        <kd  value="0"/>
+        <kd value="0"/>
     </gazebo>
     <gazebo reference="front_right_wheel_link">
@@ -124,5 +124,5 @@
         <minDepth>0.001</minDepth>
         <kp  value="10000000.0"/>
-        <kd  value="0"/>
+        <kd value="0"/>
     </gazebo>
     <gazebo reference="rear_left_wheel_link">
@@ -132,5 +132,5 @@
         <minDepth>0.001</minDepth>
         <kp  value="10000000.0"/>
-        <kd  value="0"/>
+        <kd value="0"/>
     </gazebo>
     <gazebo reference="rear_right_wheel_link">
@@ -140,5 +140,5 @@
         <minDepth>0.001</minDepth>
         <kp  value="10000000.0"/>
-        <kd  value="0"/>
+        <kd value="0"/>
     </gazebo>
 </robot>

File: limo_description/urdf/limo.xacro (robot description, xacro)
@@ -1,4 +1,4 @@
 <?xml version="1.0"?>
-<robot xmlns:xacro="http://www.ros.org/wiki/xacro" name="robot">
+<robot xmlns:xacro="http://www.ros.org/wiki/xacro" name="limo_ackerman">
     <xacro:arg name="robot_namespace" default="/" />
     <xacro:include filename="$(find limo_description)/urdf/limo_xacro.xacro" />
@@ -62,5 +62,5 @@
     <link name="rear_right_wheel_link">
         <xacro:inertial_cylinder mass="0.1" length="${wheel_length}" radius="${wheel_radius}">
-            <origin xyz="0 0 0" rpy="0 0 0"/>
+            <origin xyz="0 0 ${-wheel_length/2}" rpy="0 0 0"/>
         </xacro:inertial_cylinder>
         <visual>
@@ -81,5 +81,5 @@
     <link name="rear_left_wheel_link">
         <xacro:inertial_cylinder mass="0.1" length="${wheel_length}" radius="${wheel_radius}">
-            <origin xyz="0 0 0" rpy="0 0 0"/>
+            <origin xyz="0 0 ${wheel_length/2}" rpy="0 0 0"/>
         </xacro:inertial_cylinder>
         <visual>
@@ -100,5 +100,5 @@
     <link name="front_right_wheel_link">
         <xacro:inertial_cylinder mass="0.1" length="${wheel_length}" radius="${wheel_radius}">
-            <origin xyz="0 0 0" rpy="0 0 0"/>
+            <origin xyz="0 0 ${-wheel_length/2}" rpy="0 0 0"/>
         </xacro:inertial_cylinder>
         <visual>
@@ -119,5 +119,5 @@
     <link name="front_left_wheel_link">
         <xacro:inertial_cylinder mass="0.1" length="${wheel_length}" radius="${wheel_radius}">
-            <origin xyz="0 0 0" rpy="0 0 0"/>
+            <origin xyz="0 0 ${wheel_length/2}" rpy="0 0 0"/>
         </xacro:inertial_cylinder>
         <visual>

File: limo_description/urdf/limo_imu.xacro (robot description, xacro)
@@ -4,5 +4,5 @@
         <parent link="base_link"/>
         <child link="imu_link"/>
-        <origin xyz="0 0 0" rpy="0 0 0"/>
+        <origin xyz="0.0 0 0.1" rpy="0 0 0"/>
     </joint>
     <link name="imu_link">
@@ -26,75 +26,22 @@
         <material>Gazebo/Yellow</material>
         <sensor name="imu_sensor" type="imu">
-          <always_on>true</always_on>
-          <update_rate>100</update_rate>
-          <visualize>true</visualize>
-          <topic>__default_topic__</topic>
-          <plugin filename="libgazebo_ros_imu_sensor.so" name="imu_plugin">
-            <ros >
-                <remapping>/imu_plugin/out:=/limo/imu</remapping>
-            </ros>
-            <bodyName>imu_link</bodyName>
-            <updateRateHZ>100.0</updateRateHZ>
-            <gaussianNoise>0.001</gaussianNoise>
-            <xyzOffset>0 0 0</xyzOffset>
-            <rpyOffset>0 0 0</rpyOffset>
-            <frameName>imu_link</frameName>
-            <initialOrientationAsReference>false</initialOrientationAsReference>
-          </plugin>
-          <pose>0 0 0 0 0 0</pose>
-          <imu>
-              <angular_velocity>
-                  <x>
-                  <noise type="gaussian">
-                      <mean>0.0</mean>
-                      <stddev>2e-4</stddev>
-                      <bias_mean>0.000000</bias_mean>
-                      <bias_stddev>0.0000000</bias_stddev>
-                  </noise>
-                  </x>
-                  <y>
-                  <noise type="gaussian">
-                      <mean>0.0</mean>
-                      <stddev>2e-4</stddev>
-                      <bias_mean>0.000000</bias_mean>
-                      <bias_stddev>0.0000000</bias_stddev>
-                  </noise>
-                  </y>
-                  <z>
-                  <noise type="gaussian">
-                      <mean>0.0</mean>
-                      <stddev>2e-4</stddev>
-                      <bias_mean>0.000000</bias_mean>
-                      <bias_stddev>0.0000000</bias_stddev>
-                  </noise>
-                  </z>
-              </angular_velocity>
-              <linear_acceleration>
-                  <x>
-                  <noise type="gaussian">
-                      <mean>0.0</mean>
-                      <stddev>1.7e-2</stddev>
-                      <bias_mean>0.0</bias_mean>
-                      <bias_stddev>0.000</bias_stddev>
-                  </noise>
-                  </x>
-                  <y>
-                  <noise type="gaussian">
-                      <mean>0.0</mean>
-                      <stddev>1.7e-2</stddev>
-                      <bias_mean>0.0</bias_mean>
-                      <bias_stddev>0.000</bias_stddev>
-                  </noise>
-                  </y>
-                  <z>
-                  <noise type="gaussian">
-                      <mean>0.0</mean>
-                      <stddev>1.7e-2</stddev>
-                      <bias_mean>0.0</bias_mean>
-                      <bias_stddev>0.000</bias_stddev>
-                  </noise>
-                  </z>
-              </linear_acceleration>
-              </imu>
+            <always_on>true</always_on>
+            <update_rate>10</update_rate>
+            <visualize>true</visualize>
+            <topic>__default_topic__</topic>
+            <plugin filename="libgazebo_ros_imu_sensor.so" name="imu_plugin">
+                <ros >
+                    <remapping>/imu_plugin/out:=/limo/imu</remapping>
+                </ros>
+                <topicName>imu</topicName>
+                <bodyName>imu_link</bodyName>
+                <updateRateHZ>10.0</updateRateHZ>
+                <gaussianNoise>0.005</gaussianNoise>
+                <xyzOffset>0 0 0</xyzOffset>
+                <rpyOffset>0 0 0</rpyOffset>
+                <frame_name>imu_link</frame_name>
+                <initialOrientationAsReference>false</initialOrientationAsReference>
+            </plugin>
+            <pose>0 0 0 0 0 0</pose>
         </sensor>
     </gazebo>
