Commit message: Clean code 1

File: limo_description/urdf/gazebo.xacro (robot description, xacro)
@@ -136,38 +136,3 @@
         <kd value="0.2"/>
     </gazebo>
-    <!-- <gazebo reference="base_link">
-        <mu1>0.2</mu1>
-        <mu2>0.2</mu2>
-        <material>Gazebo/Green</material>
-    </gazebo>
-    <gazebo reference="left_steering_hinge">
-        <mu1>0.2</mu1>
-        <mu2>0.2</mu2>
-        <material>Gazebo/Green</material>
-    </gazebo>
-    <gazebo reference="right_steering_hinge">
-        <mu1>0.2</mu1>
-        <mu2>0.2</mu2>
-        <material>Gazebo/Green</material>
-    </gazebo>
-    <gazebo reference="front_left_wheel_link">
-        <mu1>0.2</mu1>
-        <mu2>0.2</mu2>
-        <material>Gazebo/Red</material>
-    </gazebo>
-    <gazebo reference="rear_left_wheel_link">
-        <mu1>0.2</mu1>
-        <mu2>0.2</mu2>
-        <material>Gazebo/Red</material>
-    </gazebo>
-    <gazebo reference="front_right_wheel_link">
-        <mu1>0.2</mu1>
-        <mu2>0.2</mu2>
-        <material>Gazebo/Blue</material>
-    </gazebo>
-    <gazebo reference="rear_right_wheel_link">
-        <mu1>0.2</mu1>
-        <mu2>0.2</mu2>
-        <material>Gazebo/Blue</material>
-    </gazebo> -->
 </robot>

File: limo_description/urdf/imu.xacro (robot description, xacro)
@@ -29,5 +29,5 @@
         <sensor name="imu_sensor" type="imu">
             <always_on>true</always_on>
-            <update_rate>10</update_rate>
+            <update_rate>100</update_rate>
             <visualize>true</visualize>
             <topic>__default_topic__</topic>
@@ -38,5 +38,5 @@
                 <topicName>imu</topicName>
                 <bodyName>imu_link</bodyName>
-                <updateRateHZ>10.0</updateRateHZ>
+                <updateRateHZ>100.0</updateRateHZ>
                 <gaussianNoise>0.005</gaussianNoise>
                 <xyzOffset>0 0 0</xyzOffset>

File: limo_description/urdf/robot.xacro (robot description, xacro)
@@ -1,7 +1,17 @@
 <?xml version="1.0"?>
-<robot xmlns:xacro="http://www.ros.org/wiki/xacro" name="ackbot">
+<robot xmlns:xacro="http://www.ros.org/wiki/xacro" name="limo_ackerman">
     <xacro:include filename="gazebo.xacro"/>
     <xacro:include filename="imu.xacro"/>
     <xacro:include filename="transmission.xacro"/>
+    <!-- Vehicle Geometries -->
+    <xacro:property name="base_x_size" value="0.2" />
+    <xacro:property name="base_y_size" value="0.13" />
+    <xacro:property name="base_z_size" value="0.1" />
+    <xacro:property name="wheelbase" value="0.2"/>
+    <xacro:property name="track" value="0.14"/>
+    <xacro:property name="base_mass" value="3.0"/>
+    <xacro:property name="wheel_vertical_offset" value="0.0" />
+    <xacro:property name="wheel_length" value="0.01" />
+    <xacro:property name="wheel_radius" value="0.045" />
     <!-- BASE LINK -->
     <link name="base_footprint">
@@ -14,5 +24,5 @@
     </joint>
     <link name="base_link">
-        <xacro:inertial_box mass="3" x="0.2" y="0.13" z="0.06">
+        <xacro:inertial_box mass="3" x="${base_x_size}" y="${base_y_size}" z="${base_z_size}">
             <origin xyz="0 0 0.025" rpy="0 0 0"/>
         </xacro:inertial_box>
@@ -20,5 +30,5 @@
             <origin xyz="0 0 0.025" rpy="0 0 0" />
             <geometry>
-                <!-- <mesh filename="file:///$(find ack_description)/meshes/Body.STL"/> -->
+                <!-- <mesh filename="file:///$(find limo_description)/meshes/limo_base.dae"/> -->
                 <box size="0.2 0.13 0.05"/>
             </geometry>
@@ -30,5 +40,5 @@
             <origin xyz="0 0 0.025" rpy="0 0 0" />
             <geometry>
-                <box size="0.2 0.13 0.06"/>
+                <box size="${base_x_size} ${base_y_size} ${base_z_size}"/>
             </geometry>
         </collision>
@@ -36,14 +46,14 @@
     <!-- WHEEL LINK -->
     <link name="rear_right_wheel_link">
-        <xacro:inertial_cylinder mass="0.1" length="0.01" radius="0.045">
-            <origin xyz="0 0 0" rpy="0 0 0"/>
-        </xacro:inertial_cylinder>
-        <visual>
-            <origin xyz="0 0 0" rpy="0 0 0" />
-            <geometry>
-                <!-- <mesh filename="file:///$(find ack_description)/meshes/Wheel.STL" /> -->
-                <cylinder radius="0.045" length="0.01"/>
-                <material name="Black">
-                    <color rgba="0 0 0 1"/>
+        <xacro:inertial_cylinder mass="0.1" length="${wheel_length}" radius="${wheel_radius}">
+            <origin xyz="0 0 0" rpy="0 0 0"/>
+        </xacro:inertial_cylinder>
+        <visual>
+            <origin xyz="0 0 0" rpy="0 0 0" />
+            <geometry>
+                <!-- <mesh filename="file:///$(find limo_description)/meshes/limo_wheel.dae" /> -->
+                <cylinder radius="${wheel_radius}" length="${wheel_length}1"/>
+                <material name="Red">
+                    <color rgba="1 0 0 1"/>
                 </material>
             </geometry>
@@ -52,20 +62,20 @@
             <origin xyz="0 0 0" rpy="0 0 0" />
             <geometry>
-                <!-- <mesh filename="file:///$(find ack_description)/meshes/Wheel.STL" /> -->
-                <cylinder radius="0.045" length="0.01"/>
+                <!-- <mesh filename="file:///$(find limo_description)/meshes/limo_wheel.dae" /> -->
+                <cylinder radius="${wheel_radius}" length="${wheel_length}"/>
             </geometry>
         </collision>
     </link>
     <link name="rear_left_wheel_link">
-        <xacro:inertial_cylinder mass="0.1" length="0.01" radius="0.045">
-            <origin xyz="0 0 0" rpy="0 0 0"/>
-        </xacro:inertial_cylinder>
-        <visual>
-            <origin xyz="0 0 0" rpy="0 0 0" />
-            <geometry>
-                <!-- <mesh filename="file:///$(find ack_description)/meshes/Wheel.STL" /> -->
-                <cylinder radius="0.045" length="0.01"/>
-                <material name="Black">
-                    <color rgba="0 0 0 1"/>
+        <xacro:inertial_cylinder mass="0.1" length="${wheel_length}" radius="${wheel_radius}">
+            <origin xyz="0 0 0" rpy="0 0 0"/>
+        </xacro:inertial_cylinder>
+        <visual>
+            <origin xyz="0 0 0" rpy="0 0 0" />
+            <geometry>
+                <!-- <mesh filename="file:///$(find limo_description)/meshes/limo_wheel.dae" /> -->
+                <cylinder radius="${wheel_radius}" length="${wheel_length}"/>
+                <material name="Red">
+                    <color rgba="1 0 0 1"/>
                 </material>
             </geometry>
@@ -74,21 +84,21 @@
             <origin xyz="0 0 0" rpy="0 0 0" />
             <geometry>
-                <!-- <mesh filename="file:///$(find ack_description)/meshes/Wheel.STL" /> -->
-                <cylinder radius="0.045" length="0.01"/>
+                <!-- <mesh filename="file:///$(find limo_description)/meshes/limo_wheel.dae" /> -->
+                <cylinder radius="${wheel_radius}" length="${wheel_length}"/>
             </geometry>
         </collision>
     </link>
     <link name="front_right_wheel_link">
-        <xacro:inertial_cylinder mass="0.1" length="0.01" radius="0.045">
-            <origin xyz="0 0 0" rpy="0 0 0"/>
-        </xacro:inertial_cylinder>
-        <visual>
-            <origin xyz="0 0 0" rpy="0 0 0" />
-            <geometry>
-                <!-- <mesh filename="file:///$(find ack_description)/meshes/Wheel.STL" /> -->
-                <cylinder radius="0.045" length="0.01"/>
-            </geometry>
-            <material name="Black">
-                <color rgba="0 0 0 1"/>
+        <xacro:inertial_cylinder mass="0.1" length="${wheel_length}" radius="${wheel_radius}">
+            <origin xyz="0 0 0" rpy="0 0 0"/>
+        </xacro:inertial_cylinder>
+        <visual>
+            <origin xyz="0 0 0" rpy="0 0 0" />
+            <geometry>
+                <!-- <mesh filename="file:///$(find limo_description)/meshes/limo_wheel.dae" /> -->
+                <cylinder radius="${wheel_radius}" length="${wheel_length}"/>
+            </geometry>
+            <material name="Red">
+                <color rgba="1 0 0 1"/>
             </material>
         </visual>
@@ -96,20 +106,20 @@
             <origin xyz="0 0 0" rpy="0 0 0" />
             <geometry>
-                <!-- <mesh filename="file:///$(find ack_description)/meshes/Wheel.STL" /> -->
-                <cylinder radius="0.045" length="0.01"/>
+                <!-- <mesh filename="file:///$(find limo_description)/meshes/limo_wheel.dae" /> -->
+                <cylinder radius="${wheel_radius}" length="${wheel_length}"/>
             </geometry>
         </collision>
     </link>
     <link name="front_left_wheel_link">
-        <xacro:inertial_cylinder mass="0.1" length="0.01" radius="0.045">
-            <origin xyz="0 0 0" rpy="0 0 0"/>
-        </xacro:inertial_cylinder>
-        <visual>
-            <origin xyz="0 0 0" rpy="0 0 0" />
-            <geometry>
-                <!-- <mesh filename="file:///$(find ack_description)/meshes/Wheel.STL" /> -->
-                <cylinder radius="0.045" length="0.01"/>
-                <material name="Black">
-                    <color rgba="0 0 0 1"/>
+        <xacro:inertial_cylinder mass="0.1" length="${wheel_length}" radius="${wheel_radius}">
+            <origin xyz="0 0 0" rpy="0 0 0"/>
+        </xacro:inertial_cylinder>
+        <visual>
+            <origin xyz="0 0 0" rpy="0 0 0" />
+            <geometry>
+                <!-- <mesh filename="file:///$(find limo_description)/meshes/limo_wheel.dae" /> -->
+                <cylinder radius="${wheel_radius}" length="${wheel_length}"/>
+                <material name="Red">
+                    <color rgba="1 0 0 1"/>
                 </material>
             </geometry>
@@ -118,16 +128,16 @@
             <origin xyz="0 0 0" rpy="0 0 0" />
             <geometry>
-                <!-- <mesh filename="file:///$(find ack_description)/meshes/Wheel.STL" /> -->
-                <cylinder radius="0.045" length="0.01"/>
+                <!-- <mesh filename="file:///$(find limo_description)/meshes/limo_wheel.dae" /> -->
+                <cylinder radius="${wheel_radius}" length="${wheel_length}"/>
             </geometry>
         </collision>
     </link>
     <link name="right_steering_hinge">
-        <xacro:inertial_flip_cylinder mass="0.1" length="0.01" radius="0.045">
+        <xacro:inertial_flip_cylinder mass="0.1" length="${wheel_length}" radius="${wheel_radius}">
             <origin xyz="0 0 0" rpy="0 0 0"/>
         </xacro:inertial_flip_cylinder>
     </link>
     <link name="left_steering_hinge">
-        <xacro:inertial_flip_cylinder mass="0.1" length="0.01" radius="0.045">
+        <xacro:inertial_flip_cylinder mass="0.1" length="${wheel_length}" radius="${wheel_radius}">
             <origin xyz="0 0 0" rpy="0 0 0"/>
         </xacro:inertial_flip_cylinder>
@@ -135,5 +145,5 @@
     <!-- WHEEL JOINT -->
     <joint name="rear_left_wheel" type="continuous">
-        <origin xyz="-0.1 0.07 0" rpy="-1.57079632679 0 0" />
+        <origin xyz="${-wheelbase/2} ${track/2} 0" rpy="-1.57079632679 0 0" />
         <parent link="base_link" />
         <child link="rear_left_wheel_link" />
@@ -147,5 +157,5 @@
     </joint>
     <joint name="rear_right_wheel" type="continuous">
-        <origin xyz="-0.1 -0.07 0" rpy="-1.57079632679 0 0" />
+        <origin xyz="${-wheelbase/2} ${-track/2} 0" rpy="-1.57079632679 0 0" />
         <parent link="base_link" />
         <child link="rear_right_wheel_link" />
@@ -159,5 +169,5 @@
     </joint>
     <joint name="left_steering_hinge_wheel" type="revolute">
-        <origin xyz="0.1 0.07 0" rpy="0 0 0" />
+        <origin xyz="${wheelbase/2} ${track/2} 0" rpy="0 0 0" />
         <parent link="base_link" />
         <child link="left_steering_hinge" />
@@ -182,5 +192,5 @@
     </joint>
     <joint name="right_steering_hinge_wheel" type="revolute">
-        <origin xyz="0.1 -0.07 0" rpy="0 0 0" />
+        <origin xyz="${wheelbase/2} ${-track/2} 0" rpy="0 0 0" />
         <parent link="base_link" />
         <child link="right_steering_hinge" />

Commit message: Update urdf

File: limo_description/urdf/gazebo.xacro (robot description, xacro)
@@ -83,5 +83,5 @@
     </gazebo>
     <gazebo reference="base_link">
-        <material>Gazebo/Red</material>
+        <material>Gazebo/White</material>
         <minDepth>0.001</minDepth>
         <kp  value="10000000.0"/>
@@ -89,5 +89,5 @@
     </gazebo>
     <gazebo reference="front_left_wheel_link">
-        <material>Gazebo/White</material>
+        <material>Gazebo/Black</material>
         <mu1>10.0</mu1>
         <mu2>10.0</mu2>
@@ -97,5 +97,5 @@
     </gazebo>
     <gazebo reference="front_right_wheel_link">
-        <material>Gazebo/White</material>
+        <material>Gazebo/Black</material>
         <mu1>10.0</mu1>
         <mu2>10.0</mu2>
@@ -105,5 +105,5 @@
     </gazebo>
     <gazebo reference="rear_left_wheel_link">
-        <material>Gazebo/White</material>
+        <material>Gazebo/Black</material>
         <mu1>10.0</mu1>
         <mu2>10.0</mu2>
@@ -113,5 +113,5 @@
     </gazebo>
     <gazebo reference="rear_right_wheel_link">
-        <material>Gazebo/White</material>
+        <material>Gazebo/Black</material>
         <mu1>10.0</mu1>
         <mu2>10.0</mu2>
@@ -121,5 +121,5 @@
     </gazebo>
     <gazebo reference="left_steering_hinge">
-        <material>Gazebo/White</material>
+        <material>Gazebo/Black</material>
         <mu1>0.1</mu1>
         <mu2>0.1</mu2>
@@ -129,5 +129,5 @@
     </gazebo>
     <gazebo reference="right_steering_hinge">
-        <material>Gazebo/White</material>
+        <material>Gazebo/Black</material>
         <mu1>0.1</mu1>
         <mu2>0.1</mu2>

File: limo_description/urdf/imu.xacro (robot description, xacro)
@@ -4,5 +4,5 @@
         <parent link="base_link"/>
         <child link="imu_link"/>
-        <origin xyz="0.0 0 0.1" rpy="0 0 0"/>
+        <origin xyz="0 0 0" rpy="0 0 0"/>
     </joint>
     <link name="imu_link">

File: limo_description/urdf/limo_meshes.xacro (robot description, xacro)
@@ -28,12 +28,8 @@
         </xacro:inertial_box>
         <visual>
-            <origin xyz="0 0 0.025" rpy="0 0 0" />
-            <geometry>
-                <!-- <mesh filename="file:///$(find limo_description)/meshes/limo_base.dae"/> -->
-                <box size="0.2 0.13 0.05"/>
-            </geometry>
-            <material name="Red">
-                <color rgba="1 0 0 1"/>
-            </material>
+            <origin xyz="0 0 ${-wheel_radius}" rpy="0 0 ${pi/2}" />
+            <geometry>
+                <mesh filename="file:///$(find limo_description)/meshes/limo_base.dae"/>
+            </geometry>
         </visual>
         <collision>
@@ -50,11 +46,7 @@
         </xacro:inertial_cylinder>
         <visual>
-            <origin xyz="0 0 0" rpy="0 0 0" />
-            <geometry>
-                <!-- <mesh filename="file:///$(find limo_description)/meshes/limo_wheel.dae" /> -->
-                <cylinder radius="${wheel_radius}" length="${wheel_length}1"/>
-                <material name="Red">
-                    <color rgba="1 0 0 1"/>
-                </material>
+            <origin xyz="0 0 0" rpy="${-pi/2} 0 0" />
+            <geometry>
+                <mesh filename="file:///$(find limo_description)/meshes/limo_wheel.dae" />
             </geometry>
         </visual>
@@ -72,11 +64,7 @@
         </xacro:inertial_cylinder>
         <visual>
-            <origin xyz="0 0 0" rpy="0 0 0" />
-            <geometry>
-                <!-- <mesh filename="file:///$(find limo_description)/meshes/limo_wheel.dae" /> -->
-                <cylinder radius="${wheel_radius}" length="${wheel_length}"/>
-                <material name="Red">
-                    <color rgba="1 0 0 1"/>
-                </material>
+            <origin xyz="0 0 0" rpy="${pi/2} 0 0" />
+            <geometry>
+                <mesh filename="file:///$(find limo_description)/meshes/limo_wheel.dae" />
             </geometry>
         </visual>
@@ -94,12 +82,8 @@
         </xacro:inertial_cylinder>
         <visual>
-            <origin xyz="0 0 0" rpy="0 0 0" />
-            <geometry>
-                <!-- <mesh filename="file:///$(find limo_description)/meshes/limo_wheel.dae" /> -->
-                <cylinder radius="${wheel_radius}" length="${wheel_length}"/>
-            </geometry>
-            <material name="Red">
-                <color rgba="1 0 0 1"/>
-            </material>
+            <origin xyz="0 0 0" rpy="${-pi/2} 0 0" />
+            <geometry>
+                <mesh filename="file:///$(find limo_description)/meshes/limo_wheel.dae" />
+            </geometry>
         </visual>
         <collision>
@@ -116,11 +100,7 @@
         </xacro:inertial_cylinder>
         <visual>
-            <origin xyz="0 0 0" rpy="0 0 0" />
-            <geometry>
-                <!-- <mesh filename="file:///$(find limo_description)/meshes/limo_wheel.dae" /> -->
-                <cylinder radius="${wheel_radius}" length="${wheel_length}"/>
-                <material name="Red">
-                    <color rgba="1 0 0 1"/>
-                </material>
+            <origin xyz="0 0 0" rpy="${pi/2} 0 0" />
+            <geometry>
+                <mesh filename="file:///$(find limo_description)/meshes/limo_wheel.dae" />
             </geometry>
         </visual>
