Commit message: Change location of odom,steer node and Update README.

File: limo_description/urdf/limo_meshes.xacro (robot description, xacro)
@@ -11,5 +11,4 @@
     <xacro:property name="track" value="0.14"/>
     <xacro:property name="base_mass" value="3.0"/>
-    <xacro:property name="wheel_vertical_offset" value="0.0" />
     <xacro:property name="wheel_length" value="0.01" />
     <xacro:property name="wheel_radius" value="0.045" />

File: limo_description/urdf/limo_no_meshes.xacro (robot description, xacro)
@@ -11,5 +11,4 @@
     <xacro:property name="track" value="0.14"/>
     <xacro:property name="base_mass" value="3.0"/>
-    <xacro:property name="wheel_vertical_offset" value="0.0" />
     <xacro:property name="wheel_length" value="0.01" />
     <xacro:property name="wheel_radius" value="0.045" />
